File: files/attiny45_led_button/attiny45_led_button.kicad_sch (KiCad schematic)
At the start: 5 parts, among them J1 Conn_02x03_Counter_Clockwise, SW1 SW_Push, U1 ATtiny45-20M

Commit message: Deployed 6b8f36f with MkDocs version: 1.6.1
Parts:
- D1: footprint Module:Carambola2 -> LED_THT:LED_D4.0mm
- J1: footprint (none) -> Connector_PinHeader_2.00mm:PinHeader_2x03_P2.00mm_Vertical
- R1: footprint (none) -> Resistor_THT:R_Axial_DIN0207_L6.3mm_D2.5mm_P7.62mm_Horizontal
- SW1: footprint (none) -> Button_Switch_THT:SW_TH_Tactile_Omron_B3F-102x
- U1: footprint Package_DFN_QFN:QFN-20-1EP_4x4mm_P0.5mm_EP2.6x2.6mm -> Package_DIP:DIP-8_W7.62mm
Changed lines of the file:
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@@
 			)
 		)
-		(property "Footprint" ""
+		(property "Footprint" "Connector_PinHeader_2.00mm:PinHeader_2x03_P2.00mm_Vertical"
 			(at 152.4 71.12 0)
 			(effects
@@
 			)
 		)
-		(property "Footprint" "Package_DFN_QFN:QFN-20-1EP_4x4mm_P0.5mm_EP2.6x2.6mm"
+		(property "Footprint" "Package_DIP:DIP-8_W7.62mm"
 			(at 106.68 85.09 0)
 			(effects
@@
 			)
 		)
-		(property "Footprint" ""
+		(property "Footprint" "Button_Switch_THT:SW_TH_Tactile_Omron_B3F-102x"
 			(at 146.05 90.17 0)
 			(effects
@@
 			)
 		)
-		(property "Footprint" "Module:Carambola2"
+		(property "Footprint" "LED_THT:LED_D4.0mm"
 			(at 125.73 63.5 0)
 			(effects
@@
 			)
 		)
-		(property "Footprint" ""
+		(property "Footprint" "Resistor_THT:R_Axial_DIN0207_L6.3mm_D2.5mm_P7.62mm_Horizontal"
 			(at 127.508 73.66 90)
 			(effects
